Commit message: feat:test

File: ros_workspace/src/zima_gazebo/robot/urdf/common_properties.urdf.xacro (robot description, xacro)
@@ -1,4 +1,5 @@
 <?xml version="1.0" ?>
-<robot name="xacro_properties" xmlns:xacro="http://ros.org/wiki/xacro">
+<robot name="xacro_properties"
+  xmlns:xacro="http://ros.org/wiki/xacro">
   <xacro:property name="M_PI" value="3.1415926535897931" />
   <material name="dark_grey">
@@ -9,18 +10,8 @@
   </material>
   <xacro:macro name="cylinder_inertia" params="mass radius height">
-    <inertia ixx="${(3*radius*radius + height*height)*mass/12}"
-             ixy="0.0"
-             ixz="0.0"
-             iyy="${(3*radius*radius + height*height)*mass/12}"
-             iyz="0.0"
-             izz="${radius*radius*mass/2}" />
+    <inertia ixx="${(3*radius*radius + height*height)*mass/12}" ixy="0.0" ixz="0.0" iyy="${(3*radius*radius + height*height)*mass/12}" iyz="0.0" izz="${radius*radius*mass/2}" />
   </xacro:macro>
   <xacro:macro name="sphere_inertia" params="mass radius">
-    <inertia ixx="${2*mass*radius*radius/5}"
-             ixy="0.0"
-             ixz="0.0"
-             iyy="${2*mass*radius*radius/5}"
-             iyz="0.0"
-             izz="${2*mass*radius*radius/5}" />
+    <inertia ixx="${2*mass*radius*radius/5}" ixy="0.0" ixz="0.0" iyy="${2*mass*radius*radius/5}" iyz="0.0" izz="${2*mass*radius*radius/5}" />
   </xacro:macro>
 </robot>

File: ros_workspace/src/zima_gazebo/robot/urdf/config.urdf.xacro (robot description, xacro)
@@ -1,75 +1,75 @@
 <?xml version="1.0"?>
 <robot xmlns:xacro="http://ros.org/wiki/xacro">
-  <xacro:property name="topic_prefix"  value="/zima_gazebo_robot"/>
-  <xacro:property name="sim_time_multi"  value="1"/>
-  <xacro:property name="chassis_radius"  value="0.175"/>
-  <xacro:property name="chassis_height"  value="0.06"/>
-  <xacro:property name="chassis_mass"  value="9"/>
-  <xacro:property name="chassis_track_length"  value="0.24"/>
-  <xacro:property name="chassis_button_distance_to_ground"  value="0.015"/>
-  <xacro:property name="chassis_bumper_update_rate"  value="50"/>
-  <xacro:property name="chassis_bumper_visualization"  value="1"/>
-  <xacro:property name="chassis_bumper_topic"  value="chassis_bumper"/>
-  <xacro:property name="chassis_odom_topic"  value="gazebo_ground_truth_odom"/>
-  <xacro:property name="chassis_odom_rate"  value="${sim_time_multi*50}"/>
-  <xacro:property name="wheel_radius"  value="0.032"/>
-  <xacro:property name="wheel_width"  value="0.02"/>
-  <xacro:property name="wheel_roll"  value="1.5707"/>
-  <xacro:property name="wheel_pitch"  value="0.0"/>
-  <xacro:property name="wheel_yaw"  value="3.1415"/>
-  <xacro:property name="wheel_mass"  value="4.85"/>
-  <xacro:property name="caster_radius"  value="${chassis_button_distance_to_ground}"/>
-  <xacro:property name="caster_mass"  value="10"/>
-  <xacro:property name="caster_x"  value="${chassis_track_length/2}"/>
-  <xacro:property name="lidar_radius"  value="0.03"/>
-  <xacro:property name="lidar_height"  value="0.03"/>
-  <xacro:property name="lidar_mass"  value="0.135"/>
-  <xacro:property name="lidar_x"  value="0.05"/>
-  <xacro:property name="lidar_y"  value="0"/>
-  <xacro:property name="lidar_z"  value="${chassis_height/2+0.01}"/>
-  <xacro:property name="lidar_yaw"  value="0"/>
-  <xacro:property name="lidar_rate"  value="${sim_time_multi*10}"/>
-  <xacro:property name="lidar_visualization"  value="0"/>
-  <xacro:property name="lidar_samples"  value="4000"/>
-  <xacro:property name="lidar_horizontal_samples"  value="${lidar_samples/lidar_rate}"/>
-  <xacro:property name="lidar_horizontal_resolution"  value="1"/>
-  <xacro:property name="lidar_horizontal_min_radian"  value="${-M_PI}"/>
-  <xacro:property name="lidar_horizontal_max_radian"  value="${M_PI}"/>
-  <xacro:property name="lidar_range_min"  value="${chassis_radius-lidar_x}"/>
-  <xacro:property name="lidar_range_max"  value="8"/>
-  <xacro:property name="lidar_range_resolution"  value="0.01"/>
-  <xacro:property name="lidar_topic"  value="lidar_scan"/>
-  <xacro:property name="lidar_bumper_topic"  value="lidar_bumper"/>
-  <xacro:property name="lidar_bumper_visualization"  value="0"/>
-  <xacro:property name="lidar_bumper_update_rate"  value="50"/>
-  <xacro:property name="left_wall_sensor_x"  value="${(chassis_radius+0.001)*0.17365}"/>
-  <xacro:property name="left_wall_sensor_y"  value="${(chassis_radius+0.001)*-0.98481}"/>
-  <xacro:property name="left_wall_sensor_z"  value="0"/>
-  <xacro:property name="left_wall_sensor_yaw"  value="-1.3963"/>
-  <xacro:property name="left_wall_sensor_rate"  value="${sim_time_multi*50}"/>
-  <xacro:property name="left_wall_sensor_visualization"  value="0"/>
-  <xacro:property name="left_wall_sensor_samples"  value="1"/>
-  <xacro:property name="left_wall_sensor_horizontal_samples"  value="${left_wall_sensor_samples}"/>
-  <xacro:property name="left_wall_sensor_horizontal_resolution"  value="1"/>
-  <xacro:property name="left_wall_sensor_horizontal_min_radian"  value="0"/>
-  <xacro:property name="left_wall_sensor_horizontal_max_radian"  value="0"/>
-  <xacro:property name="left_wall_sensor_range_min"  value="0.0005"/>
-  <xacro:property name="left_wall_sensor_range_max"  value="0.32"/>
-  <xacro:property name="left_wall_sensor_range_resolution"  value="0.001"/>
-  <xacro:property name="left_wall_sensor_topic"  value="left_wall_sensor_scan"/>
-  <xacro:property name="right_wall_sensor_x"  value="${(chassis_radius+0.001)*0.17365}"/>
-  <xacro:property name="right_wall_sensor_y"  value="${(chassis_radius+0.001)*0.98481}"/>
-  <xacro:property name="right_wall_sensor_z"  value="0"/>
-  <xacro:property name="right_wall_sensor_yaw"  value="1.3963"/>
-  <xacro:property name="right_wall_sensor_rate"  value="${sim_time_multi*50}"/>
-  <xacro:property name="right_wall_sensor_visualization"  value="0"/>
-  <xacro:property name="right_wall_sensor_samples"  value="1"/>
-  <xacro:property name="right_wall_sensor_horizontal_samples"  value="${left_wall_sensor_samples}"/>
-  <xacro:property name="right_wall_sensor_horizontal_resolution"  value="1"/>
-  <xacro:property name="right_wall_sensor_horizontal_min_radian"  value="0"/>
-  <xacro:property name="right_wall_sensor_horizontal_max_radian"  value="0"/>
-  <xacro:property name="right_wall_sensor_range_min"  value="0.0005"/>
-  <xacro:property name="right_wall_sensor_range_max"  value="0.32"/>
-  <xacro:property name="right_wall_sensor_range_resolution"  value="0.001"/>
-  <xacro:property name="right_wall_sensor_topic"  value="right_wall_sensor_scan"/>
+  <xacro:property name="topic_prefix" value="/zima_gazebo_robot"/>
+  <xacro:property name="sim_time_multi" value="1"/>
+  <xacro:property name="chassis_radius" value="0.175"/>
+  <xacro:property name="chassis_height" value="0.06"/>
+  <xacro:property name="chassis_mass" value="9"/>
+  <xacro:property name="chassis_track_length" value="0.24"/>
+  <xacro:property name="chassis_button_distance_to_ground" value="0.015"/>
+  <xacro:property name="chassis_bumper_update_rate" value="50"/>
+  <xacro:property name="chassis_bumper_visualization" value="1"/>
+  <xacro:property name="chassis_bumper_topic" value="chassis_bumper"/>
+  <xacro:property name="chassis_odom_topic" value="gazebo_ground_truth_odom"/>
+  <xacro:property name="chassis_odom_rate" value="${sim_time_multi*50}"/>
+  <xacro:property name="wheel_radius" value="0.032"/>
+  <xacro:property name="wheel_width" value="0.02"/>
+  <xacro:property name="wheel_roll" value="1.5707"/>
+  <xacro:property name="wheel_pitch" value="0.0"/>
+  <xacro:property name="wheel_yaw" value="3.1415"/>
+  <xacro:property name="wheel_mass" value="4.85"/>
+  <xacro:property name="caster_radius" value="${chassis_button_distance_to_ground}"/>
+  <xacro:property name="caster_mass" value="10"/>
+  <xacro:property name="caster_x" value="${chassis_track_length/2}"/>
+  <xacro:property name="lidar_radius" value="0.03"/>
+  <xacro:property name="lidar_height" value="0.03"/>
+  <xacro:property name="lidar_mass" value="0.135"/>
+  <xacro:property name="lidar_x" value="0.05"/>
+  <xacro:property name="lidar_y" value="0"/>
+  <xacro:property name="lidar_z" value="${chassis_height/2+0.01}"/>
+  <xacro:property name="lidar_yaw" value="0"/>
+  <xacro:property name="lidar_rate" value="${sim_time_multi*10}"/>
+  <xacro:property name="lidar_visualization" value="0"/>
+  <xacro:property name="lidar_samples" value="4000"/>
+  <xacro:property name="lidar_horizontal_samples" value="${lidar_samples/lidar_rate}"/>
+  <xacro:property name="lidar_horizontal_resolution" value="1"/>
+  <xacro:property name="lidar_horizontal_min_radian" value="${-M_PI}"/>
+  <xacro:property name="lidar_horizontal_max_radian" value="${M_PI}"/>
+  <xacro:property name="lidar_range_min" value="${chassis_radius-lidar_x}"/>
+  <xacro:property name="lidar_range_max" value="8"/>
+  <xacro:property name="lidar_range_resolution" value="0.01"/>
+  <xacro:property name="lidar_topic" value="lidar_scan"/>
+  <xacro:property name="lidar_bumper_topic" value="lidar_bumper"/>
+  <xacro:property name="lidar_bumper_visualization" value="0"/>
+  <xacro:property name="lidar_bumper_update_rate" value="50"/>
+  <xacro:property name="left_wall_sensor_x" value="${(chassis_radius+0.001)*0.17365}"/>
+  <xacro:property name="left_wall_sensor_y" value="${(chassis_radius+0.001)*-0.98481}"/>
+  <xacro:property name="left_wall_sensor_z" value="0"/>
+  <xacro:property name="left_wall_sensor_yaw" value="-1.3963"/>
+  <xacro:property name="left_wall_sensor_rate" value="${sim_time_multi*50}"/>
+  <xacro:property name="left_wall_sensor_visualization" value="0"/>
+  <xacro:property name="left_wall_sensor_samples" value="1"/>
+  <xacro:property name="left_wall_sensor_horizontal_samples" value="${left_wall_sensor_samples}"/>
+  <xacro:property name="left_wall_sensor_horizontal_resolution" value="1"/>
+  <xacro:property name="left_wall_sensor_horizontal_min_radian" value="0"/>
+  <xacro:property name="left_wall_sensor_horizontal_max_radian" value="0"/>
+  <xacro:property name="left_wall_sensor_range_min" value="0.0005"/>
+  <xacro:property name="left_wall_sensor_range_max" value="0.32"/>
+  <xacro:property name="left_wall_sensor_range_resolution" value="0.001"/>
+  <xacro:property name="left_wall_sensor_topic" value="left_wall_sensor_scan"/>
+  <xacro:property name="right_wall_sensor_x" value="${(chassis_radius+0.001)*0.17365}"/>
+  <xacro:property name="right_wall_sensor_y" value="${(chassis_radius+0.001)*0.98481}"/>
+  <xacro:property name="right_wall_sensor_z" value="0"/>
+  <xacro:property name="right_wall_sensor_yaw" value="1.3963"/>
+  <xacro:property name="right_wall_sensor_rate" value="${sim_time_multi*50}"/>
+  <xacro:property name="right_wall_sensor_visualization" value="0"/>
+  <xacro:property name="right_wall_sensor_samples" value="1"/>
+  <xacro:property name="right_wall_sensor_horizontal_samples" value="${left_wall_sensor_samples}"/>
+  <xacro:property name="right_wall_sensor_horizontal_resolution" value="1"/>
+  <xacro:property name="right_wall_sensor_horizontal_min_radian" value="0"/>
+  <xacro:property name="right_wall_sensor_horizontal_max_radian" value="0"/>
+  <xacro:property name="right_wall_sensor_range_min" value="0.0005"/>
+  <xacro:property name="right_wall_sensor_range_max" value="0.32"/>
+  <xacro:property name="right_wall_sensor_range_resolution" value="0.001"/>
+  <xacro:property name="right_wall_sensor_topic" value="right_wall_sensor_scan"/>
 </robot>

File: ros_workspace/src/zima_gazebo/robot/urdf/zima_gazebo.urdf.xacro (robot description, xacro)
@@ -1,4 +1,5 @@
 <?xml version="1.0"?>
-<robot name="zima_gazebo_robot_simulation" xmlns:xacro="http://ros.org/wiki/xacro">
+<robot name="zima_gazebo_robot_simulation"
+  xmlns:xacro="http://ros.org/wiki/xacro">
   <xacro:include filename="$(find zima_gazebo)/robot/urdf/config.urdf.xacro"/>
   <xacro:macro name="zima_gazebo_robot_sim">
@@ -78,6 +79,6 @@
       <fdir1>1.0</fdir1>
       <dynamics>
-          <damping>0.71</damping>
-          <friction>0.0</friction>
+        <damping>0.71</damping>
+        <friction>0.0</friction>
       </dynamics>
     </gazebo>
@@ -90,6 +91,6 @@
       <fdir1>1.0</fdir1>
       <dynamics>
-          <damping>0.71</damping>
-          <friction>0.0</friction>
+        <damping>0.71</damping>
+        <friction>0.0</friction>
       </dynamics>
     </gazebo>
@@ -188,23 +189,23 @@
     </gazebo>
   </xacro:macro>
-  <xacro:macro name="zima_ros_robot_controller" >
-      <gazebo>
-          <plugin name="gazebo_ros_control" filename="libgazebo_ros_control.so">
-              <legacyModeNS>true</legacyModeNS>
-              <robotSimType>gazebo_ros_control/DefaultRobotHWSim</robotSimType>
-          </plugin>
-      </gazebo>
-      <gazebo>
-          <plugin name="p3d_base_controller" filename="libgazebo_ros_p3d.so">
-              <alwaysOn>true</alwaysOn>
-              <updateRate>${chassis_odom_rate}</updateRate>
-              <bodyName>chassis_link</bodyName>
-              <topicName>${topic_prefix}/${chassis_odom_topic}</topicName>
-              <gaussianNoise>0</gaussianNoise>
-              <frameName>world</frameName>
-              <xyzOffsets>0 0 0</xyzOffsets>
-              <rpyOffsets>0 0 0</rpyOffsets>
-          </plugin>
-      </gazebo>
+  <xacro:macro name="zima_ros_robot_controller">
+    <gazebo>
+      <plugin name="gazebo_ros_control" filename="libgazebo_ros_control.so">
+        <legacyModeNS>true</legacyModeNS>
+        <robotSimType>gazebo_ros_control/DefaultRobotHWSim</robotSimType>
+      </plugin>
+    </gazebo>
+    <gazebo>
+      <plugin name="p3d_base_controller" filename="libgazebo_ros_p3d.so">
+        <alwaysOn>true</alwaysOn>
+        <updateRate>${chassis_odom_rate}</updateRate>
+        <bodyName>chassis_link</bodyName>
+        <topicName>${topic_prefix}/${chassis_odom_topic}</topicName>
+        <gaussianNoise>0</gaussianNoise>
+        <frameName>world</frameName>
+        <xyzOffsets>0 0 0</xyzOffsets>
+        <rpyOffsets>0 0 0</rpyOffsets>
+      </plugin>
+    </gazebo>
   </xacro:macro>
 </robot>

File: ros_workspace/src/zima_gazebo/robot/urdf/zima_gazebo_robot.urdf.xacro (robot description, xacro)
@@ -6,5 +6,6 @@
       zima_gazebo/launch/view_model.launch
  -->
-<robot name="zima_gazebo_robot" xmlns:xacro="http://ros.org/wiki/xacro">
+<robot name="zima_gazebo_robot"
+  xmlns:xacro="http://ros.org/wiki/xacro">
   <xacro:include filename="$(find zima_gazebo)/robot/urdf/config.urdf.xacro"/>
   <xacro:include filename="$(find zima_gazebo)/robot/urdf/common_properties.urdf.xacro"/>
@@ -35,7 +36,7 @@
     </link>
     <joint name="chassis_base_link_joint" type="fixed">
-        <origin xyz="0 0 0" rpy="0 0 0" />
-        <parent link="base_link" />
-        <child link="chassis_link" />
+      <origin xyz="0 0 0" rpy="0 0 0" />
+      <parent link="base_link" />
+      <child link="chassis_link" />
     </joint>
     <!-- left wheel -->
@@ -111,10 +112,5 @@
         <mass value="${caster_mass}" />
         <origin xyz="0 0 0" />
-        <inertia ixx="${2*caster_mass*caster_radius*caster_radius/5}"
-                 ixy="0.0"
-                 ixz="0.0"
-                 iyy="${2*caster_mass*caster_radius*caster_radius/5}"
-                 iyz="0.0"
-                 izz="${2*caster_mass*caster_radius*caster_radius/5}" />
+        <inertia ixx="${2*caster_mass*caster_radius*caster_radius/5}" ixy="0.0" ixz="0.0" iyy="${2*caster_mass*caster_radius*caster_radius/5}" iyz="0.0" izz="${2*caster_mass*caster_radius*caster_radius/5}" />
       </inertial>
     </link>
@@ -142,10 +138,5 @@
         <mass value="${caster_mass}" />
         <origin xyz="0 0 0" />
-        <inertia ixx="${2*caster_mass*caster_radius*caster_radius/5}"
-                 ixy="0.0"
-                 ixz="0.0"
-                 iyy="${2*caster_mass*caster_radius*caster_radius/5}"
-                 iyz="0.0"
-                 izz="${2*caster_mass*caster_radius*caster_radius/5}" />
+        <inertia ixx="${2*caster_mass*caster_radius*caster_radius/5}" ixy="0.0" ixz="0.0" iyy="${2*caster_mass*caster_radius*caster_radius/5}" iyz="0.0" izz="${2*caster_mass*caster_radius*caster_radius/5}" />
       </inertial>
     </link>
