Commit message: 🐞 fix(Gazebo):
修复urdf中左右沿边传感器定义错误的问题。

File: zima_gazebo/robot/urdf/config.urdf.xacro (robot description, xacro)
@@ -43,6 +43,7 @@
   <xacro:property name="lidar_bumper_visualization"  value="0"/>
   <xacro:property name="lidar_bumper_update_rate"  value="50"/>
+  <!-- 80° -->
   <xacro:property name="left_wall_sensor_x"  value="${(chassis_radius+0.001)*0.17365}"/>
-  <xacro:property name="left_wall_sensor_y"  value="${(chassis_radius+0.001)*-0.98481}"/>
+  <xacro:property name="left_wall_sensor_y"  value="${(chassis_radius+0.001)*0.98481}"/>
   <xacro:property name="left_wall_sensor_z"  value="0"/>
   <xacro:property name="left_wall_sensor_yaw"  value="-1.3963"/>
@@ -58,6 +59,7 @@
   <xacro:property name="left_wall_sensor_range_resolution"  value="0.001"/>
   <xacro:property name="left_wall_sensor_topic"  value="left_wall_sensor_scan"/>
+  <!-- -80° -->
   <xacro:property name="right_wall_sensor_x"  value="${(chassis_radius+0.001)*0.17365}"/>
-  <xacro:property name="right_wall_sensor_y"  value="${(chassis_radius+0.001)*0.98481}"/>
+  <xacro:property name="right_wall_sensor_y"  value="${(chassis_radius+0.001)*-0.98481}"/>
   <xacro:property name="right_wall_sensor_z"  value="0"/>
   <xacro:property name="right_wall_sensor_yaw"  value="1.3963"/>

Commit message: 🐞 fix(Gazebo):
修复urdf中左右沿边传感器定义错误的问题。

File: zima_gazebo/robot/urdf/config.urdf.xacro (robot description, xacro)
@@ -47,5 +47,5 @@
   <xacro:property name="left_wall_sensor_y"  value="${(chassis_radius+0.001)*0.98481}"/>
   <xacro:property name="left_wall_sensor_z"  value="0"/>
-  <xacro:property name="left_wall_sensor_yaw"  value="-1.3963"/>
+  <xacro:property name="left_wall_sensor_yaw"  value="1.3963"/>
   <xacro:property name="left_wall_sensor_rate"  value="${sim_time_multi*50}"/>
   <xacro:property name="left_wall_sensor_visualization"  value="0"/>
@@ -63,5 +63,5 @@
   <xacro:property name="right_wall_sensor_y"  value="${(chassis_radius+0.001)*-0.98481}"/>
   <xacro:property name="right_wall_sensor_z"  value="0"/>
-  <xacro:property name="right_wall_sensor_yaw"  value="1.3963"/>
+  <xacro:property name="right_wall_sensor_yaw"  value="-1.3963"/>
   <xacro:property name="right_wall_sensor_rate"  value="${sim_time_multi*50}"/>
   <xacro:property name="right_wall_sensor_visualization"  value="0"/>

Commit message: ✨ feat(悬崖传感器):
增加悬崖传感器逻辑，以及对应的仿真。

File: zima_gazebo/robot/urdf/config.urdf.xacro (robot description, xacro)
@@ -75,3 +75,67 @@
   <xacro:property name="right_wall_sensor_range_resolution"  value="0.001"/>
   <xacro:property name="right_wall_sensor_topic"  value="right_wall_sensor_scan"/>
+  <!-- 80° -->
+  <xacro:property name="left_cliff_sensor_x"  value="${(chassis_radius-0.01)*0.17365}"/>
+  <xacro:property name="left_cliff_sensor_y"  value="${(chassis_radius-0.01)*0.98481}"/>
+  <xacro:property name="left_cliff_sensor_z"  value="-${chassis_height/2}"/>
+  <xacro:property name="left_cliff_sensor_pitch"  value="1.5708"/>
+  <xacro:property name="left_cliff_sensor_rate"  value="${sim_time_multi*50}"/>
+  <xacro:property name="left_cliff_sensor_visualization"  value="1"/>
+  <xacro:property name="left_cliff_sensor_samples"  value="1"/>
+  <xacro:property name="left_cliff_sensor_horizontal_samples"  value="${left_cliff_sensor_samples}"/>
+  <xacro:property name="left_cliff_sensor_horizontal_resolution"  value="1"/>
+  <xacro:property name="left_cliff_sensor_horizontal_min_radian"  value="0"/>
+  <xacro:property name="left_cliff_sensor_horizontal_max_radian"  value="0"/>
+  <xacro:property name="left_cliff_sensor_range_min"  value="0.0005"/>
+  <xacro:property name="left_cliff_sensor_range_max"  value="0.1"/>
+  <xacro:property name="left_cliff_sensor_range_resolution"  value="0.001"/>
+  <xacro:property name="left_cliff_sensor_topic"  value="left_cliff_sensor_scan"/>
+  <!-- 15° -->
+  <xacro:property name="left_front_cliff_sensor_x"  value="${(chassis_radius-0.01)*0.96593}"/>
+  <xacro:property name="left_front_cliff_sensor_y"  value="${(chassis_radius-0.01)*0.25882}"/>
+  <xacro:property name="left_front_cliff_sensor_z"  value="-${chassis_height/2}"/>
+  <xacro:property name="left_front_cliff_sensor_pitch"  value="1.5708"/>
+  <xacro:property name="left_front_cliff_sensor_rate"  value="${sim_time_multi*50}"/>
+  <xacro:property name="left_front_cliff_sensor_visualization"  value="1"/>
+  <xacro:property name="left_front_cliff_sensor_samples"  value="1"/>
+  <xacro:property name="left_front_cliff_sensor_horizontal_samples"  value="${left_front_cliff_sensor_samples}"/>
+  <xacro:property name="left_front_cliff_sensor_horizontal_resolution"  value="1"/>
+  <xacro:property name="left_front_cliff_sensor_horizontal_min_radian"  value="0"/>
+  <xacro:property name="left_front_cliff_sensor_horizontal_max_radian"  value="0"/>
+  <xacro:property name="left_front_cliff_sensor_range_min"  value="0.0005"/>
+  <xacro:property name="left_front_cliff_sensor_range_max"  value="0.1"/>
+  <xacro:property name="left_front_cliff_sensor_range_resolution"  value="0.001"/>
+  <xacro:property name="left_front_cliff_sensor_topic"  value="left_front_cliff_sensor_scan"/>
+  <!-- -15° -->
+  <xacro:property name="right_front_cliff_sensor_x"  value="${(chassis_radius-0.01)*0.96593}"/>
+  <xacro:property name="right_front_cliff_sensor_y"  value="${(chassis_radius-0.01)*-0.25882}"/>
+  <xacro:property name="right_front_cliff_sensor_z"  value="-${chassis_height/2}"/>
+  <xacro:property name="right_front_cliff_sensor_pitch"  value="1.5708"/>
+  <xacro:property name="right_front_cliff_sensor_rate"  value="${sim_time_multi*50}"/>
+  <xacro:property name="right_front_cliff_sensor_visualization"  value="1"/>
+  <xacro:property name="right_front_cliff_sensor_samples"  value="1"/>
+  <xacro:property name="right_front_cliff_sensor_horizontal_samples"  value="${right_front_cliff_sensor_samples}"/>
+  <xacro:property name="right_front_cliff_sensor_horizontal_resolution"  value="1"/>
+  <xacro:property name="right_front_cliff_sensor_horizontal_min_radian"  value="0"/>
+  <xacro:property name="right_front_cliff_sensor_horizontal_max_radian"  value="0"/>
+  <xacro:property name="right_front_cliff_sensor_range_min"  value="0.0005"/>
+  <xacro:property name="right_front_cliff_sensor_range_max"  value="0.1"/>
+  <xacro:property name="right_front_cliff_sensor_range_resolution"  value="0.001"/>
+  <xacro:property name="right_front_cliff_sensor_topic"  value="right_front_cliff_sensor_scan"/>
+  <!-- -80° -->
+  <xacro:property name="right_cliff_sensor_x"  value="${(chassis_radius-0.01)*0.17365}"/>
+  <xacro:property name="right_cliff_sensor_y"  value="${(chassis_radius-0.01)*-0.98481}"/>
+  <xacro:property name="right_cliff_sensor_z"  value="-${chassis_height/2}"/>
+  <xacro:property name="right_cliff_sensor_pitch"  value="1.5708"/>
+  <xacro:property name="right_cliff_sensor_rate"  value="${sim_time_multi*50}"/>
+  <xacro:property name="right_cliff_sensor_visualization"  value="1"/>
+  <xacro:property name="right_cliff_sensor_samples"  value="1"/>
+  <xacro:property name="right_cliff_sensor_horizontal_samples"  value="${right_cliff_sensor_samples}"/>
+  <xacro:property name="right_cliff_sensor_horizontal_resolution"  value="1"/>
+  <xacro:property name="right_cliff_sensor_horizontal_min_radian"  value="0"/>
+  <xacro:property name="right_cliff_sensor_horizontal_max_radian"  value="0"/>
+  <xacro:property name="right_cliff_sensor_range_min"  value="0.0005"/>
+  <xacro:property name="right_cliff_sensor_range_max"  value="0.1"/>
+  <xacro:property name="right_cliff_sensor_range_resolution"  value="0.001"/>
+  <xacro:property name="right_cliff_sensor_topic"  value="right_cliff_sensor_scan"/>
 </robot>

File: zima_gazebo/robot/urdf/zima_gazebo.urdf.xacro (robot description, xacro)
@@ -187,4 +187,112 @@
       </sensor>
     </gazebo>
+    <gazebo reference="left_cliff_sensor_link">
+      <material>Gazebo/Blue</material>
+      <sensor type="ray" name="left_cliff_sensor">
+        <always_on>true</always_on>
+        <update_rate>${left_cliff_sensor_rate}</update_rate>
+        <visualize>${left_cliff_sensor_visualization}</visualize>
+        <ray>
+          <scan>
+            <horizontal>
+              <samples>${left_cliff_sensor_horizontal_samples}</samples>
+              <resolution>${left_cliff_sensor_horizontal_resolution}</resolution>
+              <min_angle>${left_cliff_sensor_horizontal_min_radian}</min_angle>
+              <max_angle>${left_cliff_sensor_horizontal_max_radian}</max_angle>
+            </horizontal>
+          </scan>
+          <range>
+            <min>${left_cliff_sensor_range_min}</min>
+            <max>${left_cliff_sensor_range_max}</max>
+            <resolution>${left_cliff_sensor_range_resolution}</resolution>
+          </range>
+        </ray>
+        <plugin name="left_cliff_sensor" filename="libgazebo_ros_laser.so">
+          <topicName>${topic_prefix}/${left_cliff_sensor_topic}</topicName>
+          <frameName>left_cliff_sensor</frameName>
+        </plugin>
+      </sensor>
+    </gazebo>
+    <gazebo reference="left_front_cliff_sensor_link">
+      <material>Gazebo/Blue</material>
+      <sensor type="ray" name="left_front_cliff_sensor">
+        <always_on>true</always_on>
+        <update_rate>${left_front_cliff_sensor_rate}</update_rate>
+        <visualize>${left_front_cliff_sensor_visualization}</visualize>
+        <ray>
+          <scan>
+            <horizontal>
+              <samples>${left_front_cliff_sensor_horizontal_samples}</samples>
+              <resolution>${left_front_cliff_sensor_horizontal_resolution}</resolution>
+              <min_angle>${left_front_cliff_sensor_horizontal_min_radian}</min_angle>
+              <max_angle>${left_front_cliff_sensor_horizontal_max_radian}</max_angle>
+            </horizontal>
+          </scan>
+          <range>
+            <min>${left_front_cliff_sensor_range_min}</min>
+            <max>${left_front_cliff_sensor_range_max}</max>
+            <resolution>${left_front_cliff_sensor_range_resolution}</resolution>
+          </range>
+        </ray>
+        <plugin name="left_front_cliff_sensor" filename="libgazebo_ros_laser.so">
+          <topicName>${topic_prefix}/${left_front_cliff_sensor_topic}</topicName>
+          <frameName>left_front_cliff_sensor</frameName>
+        </plugin>
+      </sensor>
+    </gazebo>
+    <gazebo reference="right_front_cliff_sensor_link">
+      <material>Gazebo/Blue</material>
+      <sensor type="ray" name="right_front_cliff_sensor">
+        <always_on>true</always_on>
+        <update_rate>${right_front_cliff_sensor_rate}</update_rate>
+        <visualize>${right_front_cliff_sensor_visualization}</visualize>
+        <ray>
+          <scan>
+            <horizontal>
+              <samples>${right_front_cliff_sensor_horizontal_samples}</samples>
+              <resolution>${right_front_cliff_sensor_horizontal_resolution}</resolution>
+              <min_angle>${right_front_cliff_sensor_horizontal_min_radian}</min_angle>
+              <max_angle>${right_front_cliff_sensor_horizontal_max_radian}</max_angle>
+            </horizontal>
+          </scan>
+          <range>
+            <min>${right_front_cliff_sensor_range_min}</min>
+            <max>${right_front_cliff_sensor_range_max}</max>
+            <resolution>${right_front_cliff_sensor_range_resolution}</resolution>
+          </range>
+        </ray>
+        <plugin name="right_front_cliff_sensor" filename="libgazebo_ros_laser.so">
+          <topicName>${topic_prefix}/${right_front_cliff_sensor_topic}</topicName>
+          <frameName>right_front_cliff_sensor</frameName>
+        </plugin>
+      </sensor>
+    </gazebo>
+    <gazebo reference="right_cliff_sensor_link">
+      <material>Gazebo/Blue</material>
+      <sensor type="ray" name="right_cliff_sensor">
+        <always_on>true</always_on>
+        <update_rate>${right_cliff_sensor_rate}</update_rate>
+        <visualize>${right_cliff_sensor_visualization}</visualize>
+        <ray>
+          <scan>
+            <horizontal>
+              <samples>${right_cliff_sensor_horizontal_samples}</samples>
+              <resolution>${right_cliff_sensor_horizontal_resolution}</resolution>
+              <min_angle>${right_cliff_sensor_horizontal_min_radian}</min_angle>
+              <max_angle>${right_cliff_sensor_horizontal_max_radian}</max_angle>
+            </horizontal>
+          </scan>
+          <range>
+            <min>${right_cliff_sensor_range_min}</min>
+            <max>${right_cliff_sensor_range_max}</max>
+            <resolution>${right_cliff_sensor_range_resolution}</resolution>
+          </range>
+        </ray>
+        <plugin name="right_cliff_sensor" filename="libgazebo_ros_laser.so">
+          <topicName>${topic_prefix}/${right_cliff_sensor_topic}</topicName>
+          <frameName>right_cliff_sensor</frameName>
+        </plugin>
+      </sensor>
+    </gazebo>
   </xacro:macro>
   <xacro:macro name="zima_ros_robot_controller" >

File: zima_gazebo/robot/urdf/zima_gazebo_robot.urdf.xacro (robot description, xacro)
@@ -195,4 +195,32 @@
       <child link="right_wall_sensor_link" />
     </joint>
+    <!-- left cliff sensor -->
+    <link name="left_cliff_sensor_link"/>
+    <joint name="left_cliff_sensor_joint" type="fixed">
+      <origin xyz="${left_cliff_sensor_x} ${left_cliff_sensor_y} ${left_cliff_sensor_z}" rpy="0 ${left_cliff_sensor_pitch} 0" />
+      <parent link="chassis_link"/>
+      <child link="left_cliff_sensor_link" />
+    </joint>
+    <!-- left front cliff sensor -->
+    <link name="left_front_cliff_sensor_link"/>
+    <joint name="left_front_cliff_sensor_joint" type="fixed">
+      <origin xyz="${left_front_cliff_sensor_x} ${left_front_cliff_sensor_y} ${left_front_cliff_sensor_z}" rpy="0 ${left_front_cliff_sensor_pitch} 0" />
+      <parent link="chassis_link"/>
+      <child link="left_front_cliff_sensor_link" />
+    </joint>
+    <!-- right front cliff sensor -->
+    <link name="right_front_cliff_sensor_link"/>
+    <joint name="right_front_cliff_sensor_joint" type="fixed">
+      <origin xyz="${right_front_cliff_sensor_x} ${right_front_cliff_sensor_y} ${right_front_cliff_sensor_z}" rpy="0 ${right_front_cliff_sensor_pitch} 0" />
+      <parent link="chassis_link"/>
+      <child link="right_front_cliff_sensor_link" />
+    </joint>
+    <!-- right cliff sensor -->
+    <link name="right_cliff_sensor_link"/>
+    <joint name="right_cliff_sensor_joint" type="fixed">
+      <origin xyz="${right_cliff_sensor_x} ${right_cliff_sensor_y} ${right_cliff_sensor_z}" rpy="0 ${right_cliff_sensor_pitch} 0" />
+      <parent link="chassis_link"/>
+      <child link="right_cliff_sensor_link" />
+    </joint>
     <xacro:zima_gazebo_robot_sim/>
     <xacro:zima_ros_robot_controller/>
